Commit message: Adds third link and second joint

File: two_joint_robot_description.urdf (robot description, URDF)
Before this commit: robot one_DOF_robot, 3 links, 2 joints
Links:
- added link link3, mass 1; collision cylinder length=1 radius=0.1; visual cylinder length=1 radius=0.1
Joints:
- added joint joint2: type continuous, parent link2, child link3, origin xyz=0 0 1 rpy=0 0 0, axis 0 1 0
