Commit message: Various updates

File: two_dof_robot_description.urdf (robot description, URDF)
Before this commit: robot two_DOF_robot, 4 links, 3 joints
Links:
- link link3: mass 1 -> 0.01

Commit message: Increase weight of third link

File: two_dof_robot_description.urdf (robot description, URDF)
Before this commit: robot two_DOF_robot, 4 links, 3 joints
Links:
- link link3: mass 0.01 -> 0.1
